File: schematic/esp8266-beacon.brd (EAGLE design)
At the start: 42.9 x 22.9 mm, 8 parts, among them U1 WIRELESS-WIFI-ESP-01

Commit message: Changed name from jeep to esp8266
Parts:
- added GND, GPIO2: RST, adafruit:1X01
- moved R4 2.54 mm to (33.0, 20.3)
- moved R5 2.54 mm to (33.0, 2.54)
- moved RST 2.25 mm to (11.7, 2.16)
Connections:
- new net N$1: GPIO2.1, U1.B1
- net GND: now also GND.1
Routing:
- net GND: track 87.0 -> 57.0 mm
- net N$1: track 0.00 -> 21.3 mm
- net N$5: track 38.2 -> 47.6 mm
- net 3V3: track 55.8 -> 56.4 mm
